File: board/teensyGpsDoV2/teensyGpsDoV2.kicad_sch (KiCad schematic)
At the start: 58 parts, among them J1 Screw_Terminal_01x02, J2 GPS Connector, J3 LCD_Header, J4 10MHz Out, J5 1PPS Out, SW1 SW_SPDT, U1 LM2596_Module, U2 MCP1703, U3 LT1086-5.0, U4 DAC8550, U5 74HC14, U6 Teensy4.0, U7 REF3333, X1 OSC5A2B02

Commit message: wip schematic, routing
Parts:
- SW1: footprint Connector_PinSocket_2.54mm:PinSocket_1x03_P2.54mm_Vertical -> Connector_PinHeader_2.54mm:PinHeader_1x03_P2.54mm_Vertical
Connections:
- net GND: now also J4.2 (Ext), J5.2 (Ext)
Changed lines of the file:
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@@
 	(wire
 		(pts
+			(xy 269.24 31.75) (xy 269.24 38.1)
+		)
+		(stroke
+			(width 0)
+			(type default)
+		)
+	)
+	(wire
+		(pts
 			(xy 276.86 96.52) (xy 279.4 96.52)
 		)
@@
 	(wire
 		(pts
+			(xy 190.5 45.72) (xy 191.77 45.72)
+		)
+		(stroke
+			(width 0)
+			(type default)
+		)
+	)
+	(wire
+		(pts
 			(xy 34.29 138.43) (xy 34.29 143.51)
 		)
@@
 	(wire
 		(pts
+			(xy 191.77 45.72) (xy 191.77 53.34)
+		)
+		(stroke
+			(width 0)
+			(type default)
+		)
+	)
+	(wire
+		(pts
 			(xy 130.81 31.75) (xy 133.35 31.75)
 		)
@@
 	(symbol
 		(lib_id "power:GND")
+		(at 269.24 38.1 0)
+		(unit 1)
+		(exclude_from_sim no)
+		(in_bom yes)
+		(on_board yes)
+		(dnp no)
+		(fields_autoplaced yes)
+		(property "Reference" "#PWR028"
+			(at 269.24 44.45 0)
+			(effects
+				(font
+					(size 1.27 1.27)
+				)
+				(hide yes)
+			)
+		)
+		(property "Value" "GND"
+			(at 269.24 43.18 0)
+			(effects
+				(font
+					(size 1.27 1.27)
+				)
+			)
+		)
+		(property "Footprint" ""
+			(at 269.24 38.1 0)
+			(effects
+				(font
+					(size 1.27 1.27)
+				)
+				(hide yes)
+			)
+		)
+		(property "Datasheet" ""
+			(at 269.24 38.1 0)
+			(effects
+				(font
+					(size 1.27 1.27)
+				)
+				(hide yes)
+			)
+		)
+		(property "Description" "Power symbol creates a global label with name \"GND\" , ground"
+			(at 269.24 38.1 0)
+			(effects
+				(font
+					(size 1.27 1.27)
+				)
+				(hide yes)
+			)
+		)
+		(pin "1"
+		)
+		(instances
+			(project "teensyGpsDoV2"
+				(path "/a7254994-6403-435e-b823-ccc6268898df"
+					(reference "#PWR028")
+					(unit 1)
+				)
+			)
+		)
+	)
+	(symbol
+		(lib_id "power:GND")
 		(at 74.93 55.88 0)
 		(unit 1)
@@
 			)
 		)
-		(property "Footprint" "Connector_PinSocket_2.54mm:PinSocket_1x03_P2.54mm_Vertical"
+		(property "Footprint" "Connector_PinHeader_2.54mm:PinHeader_1x03_P2.54mm_Vertical"
 			(at 223.52 111.76 0)
 			(effects
@@
 					(unit 1)
 				)
+			)
+		)
+	)
+	(symbol
+		(lib_id "power:GND")
+		(at 191.77 53.34 0)
+		(unit 1)
+		(exclude_from_sim no)
+		(in_bom yes)
+		(on_board yes)
+		(dnp no)
+		(fields_autoplaced yes)
+		(property "Reference" "#PWR029"
+			(at 191.77 59.69 0)
+			(effects
+				(font
+					(size 1.27 1.27)
+				)
+				(hide yes)
+			)
+		)
+		(property "Value" "GND"
+			(at 191.77 58.42 0)
+			(effects
+				(font
+					(size 1.27 1.27)
+				)
+			)
+		)
+		(property "Footprint" ""
+			(at 191.77 53.34 0)
+			(effects
+				(font
+					(size 1.27 1.27)
+				)
+				(hide yes)
+			)
+		)
+		(property "Datasheet" ""
+			(at 191.77 53.34 0)
+			(effects
+				(font
+					(size 1.27 1.27)
+				)
+				(hide yes)
+			)
+		)
+		(property "Description" "Power symbol creates a global label with name \"GND\" , ground"
+			(at 191.77 53.34 0)
+			(effects
+				(font
+					(size 1.27 1.27)
+				)
+				(hide yes)
+			)
+		)
+		(pin "1"
+		)
+		(instances
+			(project "teensyGpsDoV2"
+				(path "/a7254994-6403-435e-b823-ccc6268898df"
+					(reference "#PWR029")
+					(unit 1)
+				)

Commit message: schematic routing done, allegedly
Parts:
- added H5, H6, H7, H8: GPS_MountingHole, MountingHole:MountingHole_3.2mm_M3_DIN965_Pad, symbol Mechanical:MountingHole_Pad
- added J6: Conn_01x12_Pin, Connector_PinHeader_2.54mm:PinHeader_1x12_P2.54mm_Vertical, symbol Connector:Conn_01x12_Pin
- J4, J5: footprint Connector_Coaxial:SMA_Wurth_60312002114503_Vertical -> RF2-04A-T-00-50-G:CONN_RF2-04A-T-00-50-G_ADM
- U4: footprint Package_SON:VSON-8-1EP_3x3mm_P0.65mm_EP1.65x2.4mm -> Package_SO:VSSOP-8_3x3mm_P0.65mm
Connections:
- net DAC OSC VCTRL is gone; now on net DAC_OSC_VCTRL: U4.3 (V_{FB}), U4.4 (V_{OUT})
- net +3.3V: now also J2.7, J2.8, J6.11 (Pin_11), J6.2 (Pin_2); no longer J2.1, J2.2
- net GND: now also J2.2, U6.1 (GND), U6.32 (GND), H5.1, H6.1, H7.1, H8.1, J6.1 (Pin_1), J6.12 (Pin_12); no longer J2.8
- net GPS_TO_MCU_UART: now also J2.5; no longer J2.3
- net MCU_TO_GPS_UART: now also J2.3; no longer J2.5
- net at R7.2: now also J2.4; no longer J2.6
- net at U6.10 (8_TX2_IN1): now also J6.10 (Pin_10)
- net at U6.2 (0_RX1_CRX2_CS1): now also J6.3 (Pin_3)
- net at U6.3 (1_TX1_CTX2_MISO1): now also J6.4 (Pin_4)
- net at U6.4 (2_OUT2): now also J6.5 (Pin_5)
- net at U6.6 (4_BCLK2): now also J6.6 (Pin_6)
- net at U6.7 (5_IN2): now also J6.7 (Pin_7)
- net at U6.8 (6_OUT1D): now also J6.8 (Pin_8)
- net at U6.9 (7_RX2_OUT1A): now also J6.9 (Pin_9)
Other:
- note added: "Male Side, so female (this board) is mirrored 1: VDD 2: VAnt 3: TxD 4: NC 5: RxD 6: PPS 7: NC 8: GND"
- note removed: "1: VDD 2: VAnt 3: TxD 4: NC 5: RxD 6: PPS 7: NC 8: GND"
- note removed: "GPS Connector"
- moved on the sheet: FB1, J5, R10, R12, R13, R15, R4, R5, R7, U5A, U5C, U5E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
